File: Senior Design PCB v0.1/Schmatic.sch (EAGLE design)
At the start: 233 parts, among them IC1 TMC2208, IC2 TMC2208, IC3 TMC2208, IC4 TMC2208, IC5 TMC2208, IC6 CP2104, Q1 mmbt2222, Q2 mmbt2222, Q3 MMBT4403, Q4 AOD417, Q5 MMBT4403, Q6 MMBT4403, Q7 DMG3415U, U1 PCA9685, U2 AP2112-3.3, U3 HTU21DF, U4 HX711, U5 HX711, U6 HX711, X2 ESP32_WROOM32_SKINNY

Commit message: done all routing
Parts:
- removed C15, C22, C29: 0.1uF, SparkFun-Capacitors:0.1UF-25V-5%(0603)
- removed C3: 560uF, SparkFun-Capacitors:560UF-PANASONIC_G-25V-20%
- removed D3: RED, microbuilder:LED0805_NOOUTLINE
- removed R10: 1K, microbuilder:RESISTOR_0603_NOOUT
Connections:
- net EN_3 renamed EN_LIQUID_1
- net EN_4 renamed EN_LIQUID_3
- net EN_5 renamed EN_LIQUID_2
- removed net DIR_3: IC3.DIR
- removed net DIR_4: IC4.DIR
- removed net DIR_5: IC5.DIR
- removed net EN_1: IC1.ENN, R33.2
- removed net EN_2: IC2.ENN, R40.2
- removed net MS1_1: IC1.MS1
- removed net MS1_2: IC2.MS1
- removed net MS1_3: IC3.MS1
- removed net MS1_4: IC4.MS1
- removed net MS1_5: IC5.MS1
- removed net MS2_1: IC1.MS2
- removed net MS2_2: IC2.MS2
- removed net MS2_3: IC3.MS2
- removed net MS2_4: IC4.MS2
- removed net MS2_5: IC5.MS2
- removed net N$5: D3.A, R10.2
- removed net STEP_3: IC3.STEP
- removed net STEP_4: IC4.STEP
- removed net STEP_5: IC5.STEP
- removed net VDD: C15.1, C22.1, C29.1
- new net DIR_LIQUID: IC3.DIR, IC4.DIR, IC5.DIR
- new net EN_XY: IC1.ENN, IC2.ENN, R33.2, R40.2
- new net MS1_LIQUID: IC3.MS1, IC4.MS1, IC5.MS1
- new net MS1_SOLID: IC1.MS1, IC2.MS1
- new net MS2_LIQUID: IC3.MS2, IC4.MS2, IC5.MS2
- new net MS2_SOLID: IC1.MS2, IC2.MS2
- new net STEP_LIQUID: IC3.STEP, IC4.STEP, IC5.STEP
- net 5V_SERVO: no longer C3.+
- net GND: no longer C15.2, C22.2, C29.2, C3.-, D3.C
- net ONBOARD_LED: no longer R10.1
Other:
- note removed: "LED"
- moved on the sheet: C68

Commit message: update on i2c expander, fixed current pour
Parts:
- removed R3: 10k, SparkFun-Resistors:10KOHM-0603-1/10W-1%
- removed U$9: RIGHT_ANGLE_TACTILE_SWITCH, NewKevinMade:RIGHT_ANGLE_TACTILE_SWITCH
- added C15, C22, C3: 0.1uF, SparkFun-Capacitors:0.1UF-25V(+80/-20%)(0603)
- added D3: POWER, microbuilder:LED0805_NOOUTLINE
- added R10: 10K, SparkFun-Resistors:10KOHM-1/10W-1%(0603)0603
- added R90: 10k, SparkFun-Resistors:10KOHM-0603-1/10W-1%
- added RESET: KMR2, microbuilder:SWITCH_TACT_SMT4.6X2.8
- added U7: SX1509, SparkFun-DigitalIC:SX1509
- R1: value 10k -> 1K; device SparkFun-Resistors:10KOHM-0603-1/10W-1% -> microbuilder:RESISTOR_0603_NOOUT
- renumbered U$2 to WEIGHT3, U$5 to WEIGHT1, WEIGHT_SENSOR to WEIGHT2
Connections:
- removed net A0: U1.A0
- removed net A1: U1.A1
- removed net A2: U1.A2
- removed net A3: U1.A3
- removed net A4: U1.A4
- removed net A5: U1.A5
- new net !INT: U7.!INT
- new net !RESET: R10.1, U7.!RESET
- new net 10: U7.I/O[10]
- new net 11: U7.I/O[11]
- new net 15: U7.I/O[15]
- new net N$30: R90.1, U1.A0
- new net N$5: D3.A, R1.2
- new net OSCIO: U7.OSCIO
- net DIR_1: now also U7.I/O[8]
- net DIR_2: now also U7.I/O[9]
- net DIR_LIQUID: now also U7.I/O[3]
- net EN_LIQUID_1: now also U7.I/O[13]
- net EN_LIQUID_2: now also U7.I/O[14]
- net EN_LIQUID_3: now also U7.I/O[12]
- net EN_XY: now also U7.I/O[2]
- net FAN: now also U7.I/O[7]
- net GND: now also C15.2, C22.2, C3.2, D3.C, RESET.P, RESET.P1, U1.A1, U1.A2, U1.A3, U1.A4, U1.A5, U7.ADDR0, U7.ADDR1, U7.GND; no longer U$9.1, U$9.3
- net MS1_LIQUID: now also U7.I/O[4]
- net MS1_SOLID: now also U7.I/O[0]
- net MS2_LIQUID: now also U7.I/O[5]
- net MS2_SOLID: now also U7.I/O[1]
- net N$54: now also RESET.S, RESET.S1; no longer U$9.2, U$9.4
- net SCL: now also U7.SCL; no longer R3.2
- net SDA: now also U7.SDA; no longer R1.2
- net VCC: now also C15.1, C22.1, C3.1, R10.2, R90.2, U7.VCC1, U7.VCC2, U7.VDDM; no longer R3.1
- net VIB: now also U7.I/O[6]
Other:
- note added: "Allowable VCC1/2 Range: 1.2-3.6V"
- note added: "LED"
- note added: "The VCC1/2 jumpers (SJ2, SJ3) set those pins to 3.3V."
- note added: "VDD Range: 1.425-3.6V"

Commit message: added contact board
Parts:
- removed SJ1, SJ2, SJ3: JUMPER-PAD-2-NC_BY_TRACE, SparkFun-Passives:JUMPER-PAD-2-NC_BY_TRACE
Connections:
- removed net A13_I35: X2.I35/A1_7
- removed net A2_I34: X2.I34/A1_6
- removed net A5_IO4: X2.IO4/A2_0
- removed net BUZZER: X2.IO25/DAC1/A2_8
- removed net CAP_OR_BAT: X2.IO12/A2_5
- removed net CHARGE_OR_NOT: X2.IO13/A2_4
- removed net IO15_A8: X2.IO15/A2_3
- removed net IO21: X2.IO21
- removed net IO32_A7: X2.IO32/A1_4/X32P
- removed net MISO: X2.IO19
- removed net MOSI: X2.IO18
- removed net N$10: R16.1, SJ2.2, U4.DVDD, U4.RATE
- removed net N$18: R21.1, SJ1.2, U5.DVDD, U5.RATE
- removed net N$25: R26.1, SJ3.2, U6.DVDD, U6.RATE
- removed net ONBOARD_LED: X2.IO14/A2_6
- removed net RX_CUS: X2.IO27/A2_7
- removed net SCK: X2.IO5
- removed net SD_CS_MCU: X2.IO33/A1_5/X32N
- removed net TX_CUS: X2.IO26/DAC2/A2_9
- net GND: now also R16.1, R21.1, R26.1, U4.DVDD, U4.RATE, U5.DVDD, U5.RATE, U6.DVDD, U6.RATE; no longer SJ1.1, SJ2.1, SJ3.1
- net LRSW: now also X2.IO13/A2_4
- net ROTA_A: now also X2.IO21
- net ROTA_C: now also X2.IO27/A2_7
- net ROTA_E: now also X2.IO15/A2_3
- net SRSW: now also X2.IO18
- net STEP_1: now also X2.IO4/A2_0
- net STEP_2: now also X2.IO5
- net STEP_LIQUID: now also X2.IO19
- net WEIGHT_CLK_1: now also X2.IO33/A1_5/X32N
- net WEIGHT_CLK_2: now also X2.IO26/DAC2/A2_9
- net WEIGHT_CLK_3: now also X2.IO12/A2_5
- net WEIGHT_DATA_1: now also X2.IO32/A1_4/X32P
- net WEIGHT_DATA_2: now also X2.IO25/DAC1/A2_8
- net WEIGHT_DATA_3: now also X2.IO14/A2_6
- net X-HOMING: now also X2.I34/A1_6
- net Y-HOMING: now also X2.I35/A1_7
